File: Volume-AlpsRK16814MG.kicad_pcb (KiCad board)
At the start: 2 copper layers, 62.9 x 32.4 mm, 12 parts, among them J1 PWR_BR, P1 AB I/O, P2 CD I/O, P3 PWR, P4 CTRL, P5 C.G., U1 SN754410

Commit message: Changed labels on PCB and schematic so names are consistent. Readme tweak.
Parts:
- P5: value C.G. -> GND
Other:
- board text added: "+5VD"
- board text removed: "+5VDC"
Changed lines of the file:
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@@
       (effects (font (size 1.524 1.524) (thickness 0.1524)))
     )
-    (fp_text value C.G. (at -2.159 1.905) (layer F.SilkS)
+    (fp_text value GND (at -2.159 1.905) (layer F.SilkS)
       (effects (font (size 1.016 1.016) (thickness 0.2032)))
     )
@@
     (effects (font (size 1.5 1.5) (thickness 0.1524)) (justify left mirror))
   )
-  (gr_text +5VDC (at 130.81 114.554 270) (layer B.SilkS)
-    (effects (font (size 1.5 1.5) (thickness 0.1524)) (justify left mirror))
-  )
+  (gr_text +5VD (at 130.81 114.554 270) (layer B.SilkS)
+    (effects (font (size 1.5 1.5) (thickness 0.1524)) (justify left mirror))
+  )

Commit message: Initial changes for converting PCB to KiCad 5.
Parts:
- removed VAL: REF, oshw-logo-notext-100mil-FSilk
- added LOGO2: REF, oshw-logo-notext-100mil-FSilk, B.Cu at (145.9, 93.9)
- C1, C2: footprint mfk-C_4.0_2.5_2.5_0.5 -> mfk-capacitor:C_4.0_2.5_2.5_0.5
- J1: footprint mfk-SIL-2 -> mfk-connector:SIL-2
- P1, P2: footprint mfk-TE_282834-5 -> mfk-connector:TE_282834-5
- P3: footprint mfk-TE_282834-3 -> mfk-connector:TE_282834-3
- P4: footprint mfk-TE_282834-2 -> mfk-connector:TE_282834-2
- P5: footprint mfk-AVA-20ga -> mfk-1pin:AVA-20ga
- RV1: footprint mfk-ALPS_RK16814MG -> mfk-alps:ALPS_RK16814MG
- U1: footprint mfk-DIP-16_AriesC84_e -> mfk-dip:DIP-16_AriesC84_e
- renumbered VAL to LOGO1
Connections:
- RV1 pad 1: (no net) -> Net-(RV1-Pad1)
- RV1 pad 16: (no net) -> Net-(RV1-Pad16)
- RV1 pad 8: (no net) -> Net-(RV1-Pad8)
- RV1 pad 9: (no net) -> Net-(RV1-Pad9)
- U1 pad 11: (no net) -> Net-(U1-Pad11)
- U1 pad 14: (no net) -> Net-(U1-Pad14)
Other:
- outline, holes or cut-outs redrawn
- board text added: "Volume-AlpsRK16814MG v1.1"
- board text removed: "I/O"
- board text removed: "Volume-AlpsRK16814MG v1.0"

Commit message: Silk changes.
Other:
- board text added: "AB_COM"
- board text added: "CD_COM"
- board text removed: "AB_COMMON"
- board text removed: "CD_COMMON"
Changed lines of the file:
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@@
   (title_block
     (title "ALPS RK16816MG with H-bridge")
-    (date 2019-05-12)
+    (date 2019-05-14)
     (rev v1.1)
     (company "Mithat Konar")
@@
       (effects (font (size 1.524 1.524) (thickness 0.1524)))
     )
-    (fp_text value "AB I/O" (at 0 2.286) (layer Dwgs.User)
-      (effects (font (size 1.524 1.524) (thickness 0.1524)))
+    (fp_text value "AB I/O" (at 0 1.8415) (layer F.SilkS)
+      (effects (font (size 1.016 1.016) (thickness 0.1524)))
     )
     (fp_line (start 6.6 2.5) (end -6.6 2.5) (layer F.SilkS) (width 0.254))
@@
       (effects (font (size 1.524 1.524) (thickness 0.1524)))
     )
-    (fp_text value "CD I/O" (at 0 2.286) (layer Dwgs.User)
-      (effects (font (size 1.524 1.524) (thickness 0.1524)))
+    (fp_text value "CD I/O" (at 0 1.8415) (layer F.SilkS)
+      (effects (font (size 1.016 1.016) (thickness 0.1524)))
     )
     (fp_circle (center -6.6 0) (end -6.854 0) (layer F.SilkS) (width 0.254))
@@
       (effects (font (size 1.524 1.524) (thickness 0.1524)))
     )
-    (fp_text value PWR (at 0 2.286) (layer Dwgs.User)
-      (effects (font (size 1.524 1.524) (thickness 0.1524)))
+    (fp_text value PWR (at 0 1.8415) (layer F.SilkS)
+      (effects (font (size 1.016 1.016) (thickness 0.1524)))
     )
     (fp_circle (center -4.06 0) (end -4.314 0) (layer F.SilkS) (width 0.254))
@@
       (effects (font (size 1.524 1.524) (thickness 0.1524)))
     )
-    (fp_text value CTRL (at 0 2.286) (layer Dwgs.User)
-      (effects (font (size 1.524 1.524) (thickness 0.1524)))
+    (fp_text value CTRL (at 0 1.8415) (layer F.SilkS)
+      (effects (font (size 1.016 1.016) (thickness 0.1524)))
     )
     (fp_line (start 2.8 2.5) (end -2.8 2.5) (layer F.SilkS) (width 0.254))
@@
   (gr_line (start 113.665 86.995) (end 113.665 87.63) (layer Eco1.User) (width 0.1))
   (gr_text V_MOT (at 128.27 114.554 270) (layer B.SilkS)
-    (effects (font (size 1.5 1.5) (thickness 0.1524)) (justify left mirror))
+    (effects (font (size 1.016 1.016) (thickness 0.1524)) (justify left mirror))
   )
   (gr_text "Volume-AlpsRK16814MG v1.1" (at 147.32 88.265) (layer B.SilkS)
@@
   )
   (gr_text B_WIPER (at 174.625 114.554 270) (layer B.SilkS)
-    (effects (font (size 1.5 1.5) (thickness 0.1524)) (justify left mirror))
+    (effects (font (size 1.016 1.016) (thickness 0.1524)) (justify left mirror))
   )
   (gr_text B_TOP (at 172.085 114.554 270) (layer B.SilkS)
-    (effects (font (size 1.5 1.5) (thickness 0.1524)) (justify left mirror))
-  )
-  (gr_text AB_COMMON (at 169.545 114.554 270) (layer B.SilkS)
-    (effects (font (size 1.5 1.5) (thickness 0.1524)) (justify left mirror))
+    (effects (font (size 1.016 1.016) (thickness 0.1524)) (justify left mirror))
+  )
+  (gr_text AB_COM (at 169.545 114.554 270) (layer B.SilkS)
+    (effects (font (size 1.016 1.016) (thickness 0.1524)) (justify left mirror))
   )
   (gr_text A_WIPER (at 167.005 114.554 270) (layer B.SilkS)
-    (effects (font (size 1.5 1.5) (thickness 0.1524)) (justify left mirror))
+    (effects (font (size 1.016 1.016) (thickness 0.1524)) (justify left mirror))
   )
   (gr_text A_TOP (at 164.465 114.554 270) (layer B.SilkS)
-    (effects (font (size 1.5 1.5) (thickness 0.1524)) (justify left mirror))
-  )
-  (gr_text D_WIPER (at 160.655 114.554 270) (layer B.SilkS)
-    (effects (font (size 1.5 1.5) (thickness 0.1524)) (justify left mirror))
+    (effects (font (size 1.016 1.016) (thickness 0.1524)) (justify left mirror))
+  )
+  (gr_text D_WIPER (at 160.274 114.554 270) (layer B.SilkS)
+    (effects (font (size 1.016 1.016) (thickness 0.1524)) (justify left mirror))
   )
   (gr_text D_TOP (at 158.115 114.554 270) (layer B.SilkS)
-    (effects (font (size 1.5 1.5) (thickness 0.1524)) (justify left mirror))
-  )
-  (gr_text CD_COMMON (at 155.575 114.554 270) (layer B.SilkS)
-    (effects (font (size 1.5 1.5) (thickness 0.1524)) (justify left mirror))
+    (effects (font (size 1.016 1.016) (thickness 0.1524)) (justify left mirror))
+  )
+  (gr_text CD_COM (at 155.575 114.554 270) (layer B.SilkS)
+    (effects (font (size 1.016 1.016) (thickness 0.1524)) (justify left mirror))
   )
   (gr_text C_WIPER (at 153.035 114.554 270) (layer B.SilkS)
-    (effects (font (size 1.5 1.5) (thickness 0.1524)) (justify left mirror))
+    (effects (font (size 1.016 1.016) (thickness 0.1524)) (justify left mirror))
   )
   (gr_text C_TOP (at 150.495 114.554 270) (layer B.SilkS)
-    (effects (font (size 1.5 1.5) (thickness 0.1524)) (justify left mirror))
+    (effects (font (size 1.016 1.016) (thickness 0.1524)) (justify left mirror))
   )
   (gr_text "CHASSIS GND" (at 144.145 114.427 270) (layer B.SilkS)
-    (effects (font (size 1.5 1.5) (thickness 0.1524)) (justify left mirror))
+    (effects (font (size 1.016 1.016) (thickness 0.1524)) (justify left mirror))
   )
   (gr_text DGND (at 133.35 114.554 270) (layer B.SilkS)
-    (effects (font (size 1.5 1.5) (thickness 0.1524)) (justify left mirror))
+    (effects (font (size 1.016 1.016) (thickness 0.1524)) (justify left mirror))
   )
   (gr_text +5VD (at 130.81 114.554 270) (layer B.SilkS)
-    (effects (font (size 1.5 1.5) (thickness 0.1524)) (justify left mirror))
-  )
-  (gr_text VOL_DOWN (at 119.38 114.554 270) (layer B.SilkS)
-    (effects (font (size 1.5 1.5) (thickness 0.1524)) (justify left mirror))
+    (effects (font (size 1.016 1.016) (thickness 0.1524)) (justify left mirror))
+  )
+  (gr_text VOL_DOWN (at 119.253 114.554 270) (layer B.SilkS)
+    (effects (font (size 1.016 1.016) (thickness 0.1524)) (justify left mirror))
   )
   (gr_text VOL_UP (at 115.189 114.554 270) (layer B.SilkS)
-    (effects (font (size 1.5 1.5) (thickness 0.1524)) (justify left mirror))
+    (effects (font (size 1.016 1.016) (thickness 0.1524)) (justify left mirror))
   )
   (gr_text "(C) 2015 Mithat Konar" (at 141.859 113.284) (layer F.SilkS)

Commit message: Moved footprints into local archive.
Parts:
- C1, C2: footprint mfk-capacitor:C_4.0_2.5_2.5_0.5 -> Volume-AlpsRK16814MG:C_4.0_2.5_2.5_0.5
- J1: footprint mfk-connector:SIL-2 -> Volume-AlpsRK16814MG:SIL-2
- P1, P2: footprint mfk-connector:TE_282834-5 -> Volume-AlpsRK16814MG:TE_282834-5
- P3: footprint mfk-connector:TE_282834-3 -> Volume-AlpsRK16814MG:TE_282834-3
- P4: footprint mfk-connector:TE_282834-2 -> Volume-AlpsRK16814MG:TE_282834-2
- P5: footprint mfk-1pin:AVA-20ga -> Volume-AlpsRK16814MG:AVA-20ga
- RV1: footprint mfk-alps:ALPS_RK16814MG -> Volume-AlpsRK16814MG:ALPS_RK16814MG
- U1: footprint mfk-dip:DIP-16_AriesC84_e -> Volume-AlpsRK16814MG:DIP-16_AriesC84_e
