File: Volume-AlpsRK16814MG.sch (KiCad schematic (older format))
At the start: 10 parts, among them J1 PWR_BR, P1 AB I/O, P2 CD I/O, P3 PWR, P4 CTRL, P5 GND, U1 SN754410

Commit message: Initial changes for converting PCB to KiCad 5.
Parts:
- P4: footprint mfk-connector:TE_282834-3 -> mfk-connector:TE_282834-2
Changed lines of the file:
@@
 F 0 "P4" V 2700 2550 50  0000 C CNN
 F 1 "CTRL" V 2800 2550 50  0000 C CNN
-F 2 "mfk-connector:TE_282834-3" H 2750 2550 60  0001 C CNN
+F 2 "mfk-connector:TE_282834-2" H 2750 2550 60  0001 C CNN
 F 3 "" H 2750 2550 60  0000 C CNN
 	1    2750 2550

Commit message: Moved footprints into local archive.
Parts:
- C1, C2: footprint mfk-capacitor:C_4.0_2.5_2.5_0.5 -> Volume-AlpsRK16814MG:C_4.0_2.5_2.5_0.5
- J1: footprint mfk-connector:SIL-2 -> Volume-AlpsRK16814MG:SIL-2
- P1, P2: footprint mfk-connector:TE_282834-5 -> Volume-AlpsRK16814MG:TE_282834-5
- P3: footprint mfk-connector:TE_282834-3 -> Volume-AlpsRK16814MG:TE_282834-3
- P4: footprint mfk-connector:TE_282834-2 -> Volume-AlpsRK16814MG:TE_282834-2
- P5: footprint mfk-1pin:AVA-20ga -> Volume-AlpsRK16814MG:AVA-20ga
- RV1: footprint mfk-alps:ALPS_RK16814MG -> Volume-AlpsRK16814MG:ALPS_RK16814MG
- U1: footprint mfk-dip:DIP-16_AriesC84_e -> Volume-AlpsRK16814MG:DIP-16_AriesC84_e
Changed lines of the file:
@@
 Sheet 1 1
 Title "ALPS RK16816MG with H-bridge"
-Date "2019-05-12"
+Date "2019-05-15"
 Rev ""
 Comp "Mithat Konar"
@@
 F 0 "U1" H 7600 5350 60  0000 C CNN
 F 1 "SN754410" H 7600 4000 60  0000 C CNN
-F 2 "mfk-dip:DIP-16_AriesC84_e" H 7600 4650 60  0001 C CNN
+F 2 "Volume-AlpsRK16814MG:DIP-16_AriesC84_e" H 7600 4650 60  0001 C CNN
 F 3 "" H 7600 4650 60  0000 C CNN
 	1    7600 4650
@@
 F 0 "C1" H 8700 4450 40  0000 L CNN
 F 1 "100n" H 8706 4265 40  0000 L CNN
-F 2 "mfk-capacitor:C_4.0_2.5_2.5_0.5" H 8738 4200 30  0001 C CNN
+F 2 "Volume-AlpsRK16814MG:C_4.0_2.5_2.5_0.5" H 8738 4200 30  0001 C CNN
 F 3 "~" H 8700 4350 60  0000 C CNN
 	1    8700 4350
@@
 F 0 "P4" V 2700 2550 50  0000 C CNN
 F 1 "CTRL" V 2800 2550 50  0000 C CNN
-F 2 "mfk-connector:TE_282834-2" H 2750 2550 60  0001 C CNN
+F 2 "Volume-AlpsRK16814MG:TE_282834-2" H 2750 2550 60  0001 C CNN
 F 3 "" H 2750 2550 60  0000 C CNN
 	1    2750 2550
@@
 F 0 "P1" V 2700 3450 50  0000 C CNN
 F 1 "AB I/O" V 2800 3450 50  0000 C CNN
-F 2 "mfk-connector:TE_282834-5" H 2750 3450 60  0001 C CNN
+F 2 "Volume-AlpsRK16814MG:TE_282834-5" H 2750 3450 60  0001 C CNN
 F 3 "" H 2750 3450 60  0000 C CNN
 	1    2750 3450
@@
 F 0 "P2" V 2750 4800 50  0000 C CNN
 F 1 "CD I/O" V 2850 4800 50  0000 C CNN
-F 2 "mfk-connector:TE_282834-5" H 2800 4800 60  0001 C CNN
+F 2 "Volume-AlpsRK16814MG:TE_282834-5" H 2800 4800 60  0001 C CNN
 F 3 "" H 2800 4800 60  0000 C CNN
 	1    2800 4800
@@
 F 0 "RV1" H 5850 5250 50  0000 C CNN
 F 1 "RK16814MG" H 5700 3600 50  0000 C CNN
-F 2 "mfk-alps:ALPS_RK16814MG" V 4800 4900 60  0001 C CNN
+F 2 "Volume-AlpsRK16814MG:ALPS_RK16814MG" V 4800 4900 60  0001 C CNN
 F 3 "" V 4800 4900 60  0000 C CNN
 	1    4500 4500
@@
 F 0 "P5" H 5080 6150 40  0000 L CNN
 F 1 "GND" H 5000 6205 30  0001 C CNN
-F 2 "mfk-1pin:AVA-20ga" H 5000 6150 60  0001 C CNN
+F 2 "Volume-AlpsRK16814MG:AVA-20ga" H 5000 6150 60  0001 C CNN
 F 3 "" H 5000 6150 60  0000 C CNN
 	1    5000 6150
@@
 F 0 "C2" H 6850 5600 40  0000 L CNN
 F 1 "1u" H 6856 5415 40  0000 L CNN
-F 2 "mfk-capacitor:C_4.0_2.5_2.5_0.5" H 6888 5350 30  0001 C CNN
+F 2 "Volume-AlpsRK16814MG:C_4.0_2.5_2.5_0.5" H 6888 5350 30  0001 C CNN
 F 3 "TDK FK18X5R1A105K" H 6850 5500 60  0001 C CNN
 	1    6850 5500
@@
 F 0 "P3" V 2700 1800 50  0000 C CNN
 F 1 "PWR" V 2800 1800 40  0000 C CNN
-F 2 "mfk-connector:TE_282834-3" H 2750 1800 60  0001 C CNN
+F 2 "Volume-AlpsRK16814MG:TE_282834-3" H 2750 1800 60  0001 C CNN
 F 3 "" H 2750 1800 60  0000 C CNN
 	1    2750 1800
@@
 F 0 "J1" H 4750 1950 60  0000 C CNN
 F 1 "PWR_BR" H 4750 1720 40  0000 C CNN
-F 2 "mfk-connector:SIL-2" H 4750 1800 60  0001 C CNN
+F 2 "Volume-AlpsRK16814MG:SIL-2" H 4750 1800 60  0001 C CNN
 F 3 "" H 4750 1800 60  0000 C CNN
 	1    4750 1800
